Commit message: :sparkles: add tip_link to urdf

File: brio_description/urdf/brio.urdf.xacro (robot description, xacro)
@@ -73,3 +73,10 @@
         </visual>
     </link>
+    <joint name="tip_link_joint" type="fixed">
+        <origin xyz="0.2 0 0" rpy="0 0 0"/>
+        <parent link="link_4" />
+        <child link="tip_link" />
+    </joint>
+    <link name="tip_link">
+    </link>
 </robot>
